File: kicad/IoBoard/IoBoard.kicad_sch (KiCad schematic)
At the start: 18 parts, among them J1 SD Card Interface, J2 PWM, J3 Analogs, U3 MCP3208

Commit message: Component updates after first build
Parts:
- R1, R2, R3, R4, R5: value 1K -> 220R
- renumbered U3 to U1
Changed lines of the file:
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@@
       (effects (font (size 1.27 1.27)))
     )
-    (property "Value" "1K" (at 184.15 50.8 90)
+    (property "Value" "220R" (at 184.15 50.8 90)
       (effects (font (size 1.27 1.27)))
     )
@@
       (effects (font (size 1.27 1.27)))
     )
-    (property "Value" "1K" (at 184.15 33.02 90)
+    (property "Value" "220R" (at 184.15 33.02 90)
       (effects (font (size 1.27 1.27)))
     )
@@
   (symbol (lib_id "power:GND") (at 247.65 157.48 0) (unit 1)
     (in_bom yes) (on_board yes) (dnp no) (fields_autoplaced)
-    (property "Reference" "#PWR021" (at 247.65 163.83 0)
+    (property "Reference" "#PWR011" (at 247.65 163.83 0)
       (effects (font (size 1.27 1.27)) hide)
     )
@@
       (effects (font (size 1.27 1.27)))
     )
-    (property "Value" "1K" (at 184.15 41.91 90)
+    (property "Value" "220R" (at 184.15 41.91 90)
       (effects (font (size 1.27 1.27)))
     )
@@
       (effects (font (size 1.27 1.27)))
     )
-    (property "Value" "1K" (at 184.15 59.69 90)
+    (property "Value" "220R" (at 184.15 59.69 90)
       (effects (font (size 1.27 1.27)))
     )
@@
   (symbol (lib_id "power:+5V") (at 247.65 121.92 0) (unit 1)
     (in_bom yes) (on_board yes) (dnp no) (fields_autoplaced)
-    (property "Reference" "#PWR022" (at 247.65 125.73 0)
+    (property "Reference" "#PWR010" (at 247.65 125.73 0)
       (effects (font (size 1.27 1.27)) hide)
     )
@@
   (symbol (lib_id "power:+5V") (at 219.71 111.76 0) (unit 1)
     (in_bom yes) (on_board yes) (dnp no) (fields_autoplaced)
-    (property "Reference" "#PWR022" (at 219.71 115.57 0)
+    (property "Reference" "#PWR026" (at 219.71 115.57 0)
       (effects (font (size 1.27 1.27)) hide)
     )
@@
   (symbol (lib_id "Analog_ADC:MCP3208") (at 242.57 138.43 0) (unit 1)
     (in_bom yes) (on_board yes) (dnp no) (fields_autoplaced)
-    (property "Reference" "U3" (at 249.8441 123.19 0)
+    (property "Reference" "U1" (at 249.8441 123.19 0)
       (effects (font (size 1.27 1.27)) (justify left))
     )
@@
       (effects (font (size 1.27 1.27)))
     )
-    (property "Value" "1K" (at 236.22 33.02 90)
-      (effects (font (size 1.27 1.27)))
-    )
+    (property "Value" "220R" (at 236.22 33.02 90)
+      (effects (font (size 1.27 1.27)))
+    )
